File: audio_subsystems_schematics/audio_subsystems_schematics.kicad_sch (KiCad schematic)
At the start: 72 parts, among them J3 Conn_02x02_Odd_Even, J4 SWD, P1 USB_C_Plug_USB2.0, SW1 BOOTSEL, SW2 RESET, U1 RP2040, U2 TAS5805MPWP, U3 TC2014-3.3VxCTTR, U4 W25Q16JV, Y1 Crystal_GND2_Small

Commit message: Power amp PVDD directly from VBUS
Remove ferrite bead FB2 and the PVDD decoupling caps C30-C33; the
TAS5805M PVDD pins now sit on VBUS with a 47 uF bulk cap (C39).
No RP2040 pin assignments change.

Drop KiCad lock and autosave files from the repo and ignore them,
and add the latest KiCad backup.

Co-Authored-By: Claude Opus 5.5 <noreply@anthropic.com>
Parts:
- removed C30, C31: 47uF, symbol Device:C_Small
- removed C32, C33: 1uF, symbol Device:C_Small
- removed FB2: Ferrite bead, symbol Device:FerriteBead_Small
- added C39: 47uF, symbol Device:C_Small
Connections:
- net PVDD is gone; now on net VBUS: U2.15 (PVDD), U2.16 (PVDD), U2.27 (PVDD), U2.28 (PVDD)
- net GNDREF: now also C39.2
- net VBUS: now also C39.1
Other:
- note removed: "Amp PVDD supply (from USB 5V) and decoupling"
- note removed: "Amp regulator and digital supply caps"
- moved on the sheet: C34, C35, C36, C37, C38, R11
